File: SmartTagPrototype.kicad_sch (KiCad schematic)
At the start: 48 parts, among them IC1 NRF52810-QFAA-R7, IC3 AEM30940-QFN, J1 Connection pins for AC / ante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, J2 SWD Connection Pins, J3 UART, J4 Port 11 - 18, J5 Port 0 - 5, J6 Port 22- 24, X1 32MHz

Commit message: dodanie footprintow do kondensatorow
Parts:
- C1, C5, C8: footprint Capacitor_SMD:C_0201_0603Metric -> Capacitor_THT:CP_Radial_D5.0mm_P2.50mm
- C3: footprint Capacitor_SMD:C_0201_0603Metric -> Library:C_2.8x1
- C4: footprint CAPC1005X61N -> Capacitor_THT:CP_Radial_D5.0mm_P2.50mm
- C7: footprint CAPC0603X33N -> Capacitor_THT:CP_Radial_D5.0mm_P2.50mm
- C9: footprint CAPC1608X90N -> Capacitor_THT:CP_Radial_D4.0mm_P2.00mm
- CBUCK1, CHV1, CLV1, CSRC1: footprint CAPC0603X33N -> Capacitor_THT:CP_Radial_D4.0mm_P2.00mm
- CX1, CX2: footprint CAPC1608X90N -> Library:C_2.8x1
- D10, D11, D12, D13: footprint (none) -> Diode_SMD:D_SOD-323F
- PHVL-3R9H474-R1, PHVL-3R9H474-R2: footprint Capacitor_THT:C_Rect_L16.5mm_W9.0mm_P15.00mm_MKT -> Capacitor_THT:CP_Radial_D5.0mm_P2.50mm
Changed lines of the file:
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@@
 			)
 		)
-		(property "Footprint" "CAPC0603X33N"
+		(property "Footprint" "Capacitor_THT:CP_Radial_D4.0mm_P2.00mm"
 			(at 27 137.16 0)
 			(effects
@@
 			)
 		)
-		(property "Footprint" ""
+		(property "Footprint" "Diode_SMD:D_SOD-323F"
 			(at 132.08 49.53 0)
 			(effects
@@
 			)
 		)
-		(property "Footprint" "CAPC0603X33N"
+		(property "Footprint" "Capacitor_THT:CP_Radial_D4.0mm_P2.00mm"
 			(at 93.98 -56.82 0)
 			(effects
@@
 			)
 		)
-		(property "Footprint" "Capacitor_SMD:C_0201_0603Metric"
+		(property "Footprint" "Capacitor_THT:CP_Radial_D5.0mm_P2.50mm"
 			(at 194.0052 58.42 0)
 			(effects
@@
 			)
 		)
-		(property "Footprint" "Capacitor_THT:C_Rect_L16.5mm_W9.0mm_P15.00mm_MKT"
+		(property "Footprint" "Capacitor_THT:CP_Radial_D5.0mm_P2.50mm"
 			(at 147.32 115.57 0)
 			(effects
@@
 			)
 		)
-		(property "Footprint" ""
+		(property "Footprint" "Diode_SMD:D_SOD-323F"
 			(at 132.08 39.37 0)
 			(effects
@@
 			)
 		)
-		(property "Footprint" "CAPC1608X90N"
+		(property "Footprint" "Library:C_2.8x1"
 			(at 259.08 149.53 0)
 			(effects
@@
 			)
 		)
-		(property "Footprint" ""
+		(property "Footprint" "Diode_SMD:D_SOD-323F"
 			(at 119.38 49.53 0)
 			(effects
@@
 			)
 		)
-		(property "Footprint" "CAPC0603X33N"
+		(property "Footprint" "Capacitor_THT:CP_Radial_D5.0mm_P2.50mm"
 			(at 166.7 102.87 0)
 			(effects
@@
 			)
 		)
-		(property "Footprint" "Capacitor_THT:C_Rect_L16.5mm_W9.0mm_P15.00mm_MKT"
+		(property "Footprint" "Capacitor_THT:CP_Radial_D5.0mm_P2.50mm"
 			(at 139.7 101.6 0)
 			(effects
@@
 			)
 		)
-		(property "Footprint" "Capacitor_SMD:C_0201_0603Metric"
+		(property "Footprint" "Capacitor_THT:CP_Radial_D5.0mm_P2.50mm"
 			(at 232.1052 80.01 0)
 			(effects
@@
 			)
 		)
-		(property "Footprint" "CAPC1005X61N"
+		(property "Footprint" "Capacitor_THT:CP_Radial_D5.0mm_P2.50mm"
 			(at 270.18 76.2 0)
 			(effects
@@
 			)
 		)
-		(property "Footprint" "Capacitor_SMD:C_0201_0603Metric"
+		(property "Footprint" "Capacitor_THT:CP_Radial_D5.0mm_P2.50mm"
 			(at 182.5752 147.32 0)
 			(effects
@@
 			)
 		)
-		(property "Footprint" "CAPC0603X33N"
+		(property "Footprint" "Capacitor_THT:CP_Radial_D4.0mm_P2.00mm"
 			(at 19.38 137.16 0)
 			(effects
@@
 			)
 		)
-		(property "Footprint" ""
+		(property "Footprint" "Diode_SMD:D_SOD-323F"
 			(at 119.38 39.37 0)
 			(effects
@@
 			)
 		)
-		(property "Footprint" "Capacitor_SMD:C_0201_0603Metric"
+		(property "Footprint" "Library:C_2.8x1"
 			(at 243.5352 107.95 0)
 			(effects
@@
 			)
 		)
-		(property "Footprint" "CAPC1608X90N"
+		(property "Footprint" "Library:C_2.8x1"
 			(at 259.08 186.36 0)
 			(effects
@@
 			)
 		)
-		(property "Footprint" "CAPC0603X33N"
+		(property "Footprint" "Capacitor_THT:CP_Radial_D4.0mm_P2.00mm"
 			(at 58.42 -4.75 0)
 			(effects
@@
 			)
 		)
-		(property "Footprint" "CAPC1608X90N"
+		(property "Footprint" "Capacitor_THT:CP_Radial_D4.0mm_P2.00mm"
 			(at 284.15 48.26 0)
 			(effects

Commit message: Updated sch
Parts:
- removed AE2: Antenna, RF_Antenna:Astrocast_AST50127-00, symbol Device:Antenna
- removed J1: Connection pins for AC / antenna, symbol Connector:Conn_01x02_Pin
- removed J5: Port 0 - 5, symbol Connector:Conn_01x06_Pin
- added J1: Nordic output antenna, symbol Connector:Conn_Coaxial
- added J10: SWD, symbol Connector:Conn_01x04_Pin
- added J11: Port 9 -10, symbol Connector:Conn_01x02_Pin
- added J12: Port 0 - 5, symbol Connector:Conn_01x06_Pin
- added J7: Additional AC pins, symbol Connector:Conn_01x02_Pin
- added J8: Conn_Coaxial, symbol Connector:Conn_Coaxial
- added J9: AC pins (generator/antenna), symbol Connector:Conn_01x02_Pin
- added R15, R16, R17, R18: 0, symbol Device:R_Small
- J2: value SWD Connection Pins -> Capacitor Voltage
Connections:
- net GND: now also J2.2 (Pin_2), J1.2 (Ext), J10.4 (Pin_4)
- net VBUCK: now also R15.1, R16.1, R17.1
- net at IC1.2 (P0.00/XL1): now also J12.1 (Pin_1)
- net at IC1.3 (P0.01/XL2): now also J12.2 (Pin_2)
- net at IC1.4 (P0.02/AIN0): now also J12.3 (Pin_3)
- net at IC1.5 (P0.03/AIN1): now also J12.4 (Pin_4)
- net at IC1.6 (P0.04/AIN2): now also J12.5 (Pin_5)
- net at IC1.7 (P0.05/AIN3): now also J12.6 (Pin_6)
- net at D11.2 (A), D13.1 (K), R12.1: now also R1.1, R18.2
- net at R6.2: now also IC3.6 (CFG[0]), R17.2
- net at D10.2 (A), D12.1 (K), R13.1: now also R2.1, R3.2
- net at R4.2: now also IC3.4 (CFG[2]), R15.2
- net at IC3.5 (CFG[1]): now also R5.2, R16.2; no longer R2.2
- net at R13.2: now also J8.2 (Ext)
- net at L1.2: now also J1.1 (In)
- net at R12.2: now also J8.1 (In)
- net at IC1.11 (P0.09): now also J11.1 (Pin_1)
- net at IC1.12 (P0.10): now also J11.2 (Pin_2)
- net at IC1.24 (P0.21/NRESET): now also J10.1 (Pin_1)
- net at J2.1 (Pin_1): now also IC3.16 (BATT), PHVL-3R9H474-R1.1; no longer IC1.25 (SWDCLK)
- net at IC1.26 (SWDIO): now also J10.3 (Pin_3); no longer J2.2 (Pin_2)
- net at R3.1: now also J9.2 (Pin_2)
- net at R1.2: now also J7.1 (Pin_1); no longer IC3.4 (CFG[2])
- new net: J9.1 (Pin_1), R18.1
- new net: J7.2 (Pin_2), R2.2
- new net: IC1.25 (SWDCLK), J10.2 (Pin_2)
Other:
- note added: "+"
- note added: "-"
- note added: "GND"
- note added: "One AC source at a time!"
- note added: "RESET"
- moved on the sheet: C7, CHV1, CLV1
