File: SmartTagPrototype.kicad_sch (KiCad schematic)
At the start: 56 parts, among them IC1 NRF52810-QFAA-R7, IC3 AEM30940-QFN, J1 Nordic output antenna, J10 SWD, J11 Port 9 -10, J12 Port 0 - 5, J2 Capacitor Voltage, J3 UART, J4 Port 11 - 18, J6 Port 22- 24, J7 Additional AC pins, J8 Conn_Coaxial, J9 AC pins (generator/antenna), X1 32MHz

Commit message: dodane gniazda i rezystory, cewki ciagle do zrobienia
Parts:
- J1, J8: footprint (none) -> Library:U_FL
- R1, R10, R11, R12, R13, R14, R15, R16, R17, R18, R2, R3, R4, R5, R6, R7, R8, R9: footprint (none) -> Jumper:SolderJumper-2_P1.3mm_Open_TrianglePad1.0x1.5mm
Changed lines of the file:
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@@
 	(label "VBUCK"
 		(at 69.85 62.23 0)
+		(fields_autoplaced yes)
 		(effects
 			(font
@@
 	(label "VBUCK"
 		(at 83.82 104.14 0)
+		(fields_autoplaced yes)
 		(effects
 			(font
@@
 			)
 		)
-		(property "Footprint" ""
+		(property "Footprint" "Jumper:SolderJumper-2_P1.3mm_Open_TrianglePad1.0x1.5mm"
 			(at 67.31 109.22 0)
 			(effects
@@
 			)
 		)
-		(property "Footprint" ""
+		(property "Footprint" "Library:U_FL"
 			(at 252.73 134.62 0)
 			(effects
@@
 			)
 		)
-		(property "Footprint" ""
+		(property "Footprint" "Jumper:SolderJumper-2_P1.3mm_Open_TrianglePad1.0x1.5mm"
 			(at 139.7 115.57 0)
 			(effects
@@
 			)
 		)
-		(property "Footprint" ""
+		(property "Footprint" "Jumper:SolderJumper-2_P1.3mm_Open_TrianglePad1.0x1.5mm"
 			(at 132.08 30.48 0)
 			(effects
@@
 			)
 		)
-		(property "Footprint" ""
+		(property "Footprint" "Jumper:SolderJumper-2_P1.3mm_Open_TrianglePad1.0x1.5mm"
 			(at 245.11 95.25 0)
 			(effects
@@
 			)
 		)
-		(property "Footprint" ""
+		(property "Footprint" "Jumper:SolderJumper-2_P1.3mm_Open_TrianglePad1.0x1.5mm"
 			(at 80.01 109.22 0)
 			(effects
@@
 			)
 		)
-		(property "Footprint" ""
+		(property "Footprint" "Jumper:SolderJumper-2_P1.3mm_Open_TrianglePad1.0x1.5mm"
 			(at 133.35 105.41 0)
 			(effects
@@
 			)
 		)
-		(property "Footprint" ""
+		(property "Footprint" "Library:U_FL"
 			(at 124.46 13.97 0)
 			(effects
@@
 			)
 		)
-		(property "Footprint" ""
+		(property "Footprint" "Jumper:SolderJumper-2_P1.3mm_Open_TrianglePad1.0x1.5mm"
 			(at 132.08 27.94 0)
 			(effects
@@
 			)
 		)
-		(property "Footprint" ""
+		(property "Footprint" "Jumper:SolderJumper-2_P1.3mm_Open_TrianglePad1.0x1.5mm"
 			(at 120.65 29.21 0)
 			(effects
@@
 			)
 		)
-		(property "Footprint" ""
+		(property "Footprint" "Jumper:SolderJumper-2_P1.3mm_Open_TrianglePad1.0x1.5mm"
 			(at 80.01 111.76 0)
 			(effects
@@
 			)
 		)
-		(property "Footprint" ""
+		(property "Footprint" "Jumper:SolderJumper-2_P1.3mm_Open_TrianglePad1.0x1.5mm"
 			(at 127 22.86 0)
 			(effects
@@
 			)
 		)
-		(property "Footprint" ""
+		(property "Footprint" "Jumper:SolderJumper-2_P1.3mm_Open_TrianglePad1.0x1.5mm"
 			(at 124.46 22.86 0)
 			(effects
@@
 			)
 		)
-		(property "Footprint" ""
+		(property "Footprint" "Jumper:SolderJumper-2_P1.3mm_Open_TrianglePad1.0x1.5mm"
 			(at 144.78 110.49 0)
 			(effects
@@
 			)
 		)
-		(property "Footprint" ""
+		(property "Footprint" "Jumper:SolderJumper-2_P1.3mm_Open_TrianglePad1.0x1.5mm"
 			(at 238.76 90.17 0)
 			(effects
@@
 			)
 		)
-		(property "Footprint" ""
+		(property "Footprint" "Jumper:SolderJumper-2_P1.3mm_Open_TrianglePad1.0x1.5mm"
 			(at 67.31 106.68 0)
 			(effects
@@
 			)
 		)
-		(property "Footprint" ""
+		(property "Footprint" "Jumper:SolderJumper-2_P1.3mm_Open_TrianglePad1.0x1.5mm"
 			(at 67.31 111.76 0)
 			(effects
@@
 			)
 		)
-		(property "Footprint" ""
+		(property "Footprint" "Jumper:SolderJumper-2_P1.3mm_Open_TrianglePad1.0x1.5mm"
 			(at 238.76 87.63 0)
 			(effects
@@
 			)
 		)
-		(property "Footprint" ""
+		(property "Footprint" "Jumper:SolderJumper-2_P1.3mm_Open_TrianglePad1.0x1.5mm"
 			(at 120.65 26.67 0)
 			(effects
@@
 			)
 		)
-		(property "Footprint" ""
+		(property "Footprint" "Jumper:SolderJumper-2_P1.3mm_Open_TrianglePad1.0x1.5mm"
 			(at 80.01 106.68 0)
 			(effects

Commit message: dobra, dodalem cewki. Ide spac
Parts:
- L1: footprint LQW18AS10NG0CD -> Library:SMD_2.0x1.0
- LBOOST1: footprint LQM18DH330M70L -> Library:SMD_1.6_1.5
- LBUCK1: footprint Library:JELF243A -> Library:SMD_1.6_1.5
Changed lines of the file:
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@@
 			)
 		)
-		(property "Footprint" "Library:JELF243A"
+		(property "Footprint" "Library:SMD_1.6_1.5"
 			(at 74.93 -7.29 0)
 			(effects
@@
 			)
 		)
-		(property "Footprint" "LQW18AS10NG0CD"
+		(property "Footprint" "Library:SMD_2.0x1.0"
 			(at 156.54 116.84 0)
 			(effects
@@
 			)
 		)
-		(property "Footprint" "LQM18DH330M70L"
+		(property "Footprint" "Library:SMD_1.6_1.5"
 			(at 200.33 44.45 0)
 			(effects

Commit message: jeszcze kondensator zgubilem, teraz jest WSZYSTKO (punkty testowe kiedy indziej sie zrobi)
Parts:
- CBOOST1: footprint CAPC1608X90N -> Capacitor_THT:CP_Radial_D4.0mm_P2.00mm
Changed lines of the file:
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@@
 			)
 		)
-		(property "Footprint" "CAPC1608X90N"
+		(property "Footprint" "Capacitor_THT:CP_Radial_D4.0mm_P2.00mm"
 			(at 185.09 76.2 0)
 			(effects

Commit message: wstępnie poukładane pcb
Other:
- note removed: "NIE WIEM JAKA OBUDOWA DO TEGO UKŁADU footprinty są na obydwie, możecie przełączyć w razie czego"
Changed lines of the file:
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@@
-		)
-	)
-	(text "NIE WIEM JAKA OBUDOWA DO TEGO UKŁADU\nfootprinty są na obydwie, możecie przełączyć w razie czego"
-		(exclude_from_sim no)
-		(at 200.66 81.788 0)
-		(effects
-			(font
-				(size 1.27 1.27)
-			)
 		)
 	)
@@
 		)
 	)
-	(text "-"
-		(exclude_from_sim no)
-		(at 131.318 28.194 0)
-		(effects
-			(font
-				(size 1.27 1.27)
-			)
-		)
-	)
 	(text "SWDIO"
 		(exclude_from_sim no)
@@
 	(label "VBUCK"
 		(at 69.85 62.23 0)
-		(fields_autoplaced yes)
 		(effects
 			(font
@@
 	(label "VBUCK"
 		(at 83.82 104.14 0)
-		(fields_autoplaced yes)
 		(effects
 			(font

Commit message: push abominacji czytaj dodany footprint i symbol zlacza testowego (niech Bog ma mnie w opiece)
Parts:
- removed J10: SWD, symbol Connector:Conn_01x04_Pin
- removed J11: Port 9 -10, symbol Connector:Conn_01x02_Pin
- removed J12: Port 0 - 5, symbol Connector:Conn_01x06_Pin
- removed J2: Capacitor Voltage, symbol Connector:Conn_01x02_Pin
- removed J3: UART, symbol Connector:Conn_01x02_Pin
- removed J4: Port 11 - 18, symbol Connector:Conn_01x08_Pin
- removed J6: Port 22- 24, symbol Connector:Conn_01x03_Pin
- added DIAG1: ~, Library:DIAG, symbol Library:Diag
- J7, J9: footprint (none) -> Connector_PinHeader_2.54mm:PinHeader_1x02_P2.54mm_Vertical
Connections:
- net GND: now also DIAG1.0 (C_vol_GND), DIAG1.15 (GND), DIAG1.19 (GND)
- net at IC1.22 (P0.19): now also DIAG1.24 (Port_19_TX)
- net at IC1.23 (P0.20): now also DIAG1.23 (Port_20_RX)
- net at IC1.11 (P0.09): now also DIAG1.7 (Port_9)
- net at IC1.12 (P0.10): now also DIAG1.8 (Port_10)
- net at IC1.2 (P0.00/XL1): now also DIAG1.1 (Port_0)
- net at IC1.3 (P0.01/XL2): now also DIAG1.2 (Port_1)
- net at IC1.4 (P0.02/AIN0): now also DIAG1.3 (Port_2)
- net at IC1.5 (P0.03/AIN1): now also DIAG1.4 (Port_3)
- net at IC1.6 (P0.04/AIN2): now also DIAG1.5 (Port_4)
- net at IC1.7 (P0.05/AIN3): now also DIAG1.6 (Port_5)
- net at IC3.16 (BATT), PHVL-3R9H474-R1.1: now also DIAG1.14 (C_vol_VCC)
- net at IC1.14 (P0.11): now also DIAG1.9 (Port_11)
- net at IC1.15 (P0.12): now also DIAG1.10 (Port_12)
- net at IC1.16 (P0.13): now also DIAG1.11 (Port_13)
- net at IC1.17 (P0.14): now also DIAG1.12 (Port_14)
- net at IC1.18 (P0.15): now also DIAG1.13 (Port_15)
- net at IC1.19 (P0.16): now also DIAG1.27 (Port_16)
- net at IC1.20 (P0.17): now also DIAG1.26 (Port_17)
- net at IC1.21 (P0.18): now also DIAG1.25 (Port_18)
- net at IC1.24 (P0.21/NRESET): now also DIAG1.22 (Port_21_RESET)
- net at IC1.25 (SWDCLK): now also DIAG1.21 (Port_25_SWDCLK)
- net at IC1.26 (SWDIO): now also DIAG1.20 (Port_26_SWDIO)
- net at IC1.27 (P0.22): now also DIAG1.18 (Port_22)
- net at IC1.28 (P0.23): now also DIAG1.17 (Port_23)
- net at IC1.29 (P0.24): now also DIAG1.16 (Port_24)
Other:
- note removed: "+"
- note removed: "-"
- note removed: "RX"
- note removed: "TX"
